Commit message: 更新脚踝数据

File: X1无皮肤版本/X1.urdf (robot description, URDF)
Before this commit: robot X1, 26 links, 25 joints
Links:
- link left_ankle_pitch_link: mass 0.1957028 -> 0.34756029
- link right_ankle_pitch_link: mass 0.2755193 -> 0.34756014

File: X1有皮肤版本/X1.urdf (robot description, URDF)
Before this commit: robot X1, 26 links, 25 joints
Links:
- link left_ankle_pitch_link: mass 0.1957028 -> 0.34756029
- link right_ankle_pitch_link: mass 0.2755193 -> 0.34756014
