Commit message: 更新无皮肤版本的参数,优化了碰撞体与文件结构

File: x1_with_skin/urdf/X1.urdf (robot description, URDF)
Before this commit: robot X1, 26 links, 25 joints
Links:
- link head_link: geometry collision sphere radius=0.0621; visual mesh filename=../meshes/head_link.STL
- link left_ankle_pitch_link: geometry collision sphere radius=0.035; visual mesh filename=../meshes/left_ankle_pitch_link.STL
- link left_ankle_roll_link: geometry collision sphere radius=0.01; collision sphere radius=0.01
- link left_elbow_link: geometry collision cylinder length=0.08 radius=0.02; visual mesh filename=../meshes/left_elbow_link.STL
- link left_hand_roll_link: geometry collision cylinder length=0.2 radius=0.02; visual mesh filename=../meshes/left_hand_roll_link.STL
- link left_hip_pitch_link: geometry collision cylinder length=0.3 radius=0.05; visual mesh filename=../meshes/left_hip_pitch_link.STL
- link left_hip_roll_link: geometry collision sphere radius=0.04; visual mesh filename=../meshes/left_hip_roll_link.STL
- link left_hip_yaw_link: geometry collision sphere radius=0.05; visual mesh filename=../meshes/left_hip_yaw_link.STL
- link left_knee_link: geometry collision cylinder length=0.25 radius=0.05; visual mesh filename=../meshes/left_knee_link.STL
- link left_shoulder_pitch_link: geometry collision sphere radius=0.025; visual mesh filename=../meshes/left_shoulder_pitch_link.STL
- link left_shoulder_roll_link: geometry collision cylinder length=0.1 radius=0.02; visual mesh filename=../meshes/left_shoulder_roll_link.STL
- link left_shoulder_yaw_link: geometry collision cylinder length=0.07 radius=0.02; visual mesh filename=../meshes/left_shoulder_yaw_link.STL
- link pelvis_link: geometry visual mesh filename=../meshes/pelvis_link.STL
- link right_ankle_pitch_link: geometry collision sphere radius=0.035; visual mesh filename=../meshes/right_ankle_pitch_link.STL
- link right_ankle_roll_link: geometry collision sphere radius=0.01; collision sphere radius=0.01
- link right_elbow_link: geometry collision cylinder length=0.08 radius=0.02; visual mesh filename=../meshes/right_elbow_link.STL
- link right_hand_roll_link: geometry collision cylinder length=0.2 radius=0.02; visual mesh filename=../meshes/right_hand_roll_link.STL
- link right_hip_pitch_link: geometry collision cylinder length=0.3 radius=0.05; visual mesh filename=../meshes/right_hip_pitch_link.STL
- link right_hip_roll_link: geometry collision sphere radius=0.04; visual mesh filename=../meshes/right_hip_roll_link.STL
- link right_hip_yaw_link: geometry collision sphere radius=0.05; visual mesh filename=../meshes/right_hip_yaw_link.STL
- link right_knee_link: geometry collision cylinder length=0.25 radius=0.05; visual mesh filename=../meshes/right_knee_link.STL
- link right_shoulder_pitch_link: geometry collision sphere radius=0.025; visual mesh filename=../meshes/right_shoulder_pitch_link.STL
- link right_shoulder_roll_link: geometry collision cylinder length=0.1 radius=0.02; visual mesh filename=../meshes/right_shoulder_roll_link.STL
- link right_shoulder_yaw_link: geometry collision cylinder length=0.07 radius=0.02; visual mesh filename=../meshes/right_shoulder_yaw_link.STL
- link torso_link: geometry collision cylinder length=0.3 radius=0.1; visual mesh filename=../meshes/torso_link.STL
- link waist_yaw_link: geometry visual mesh filename=../meshes/waist_yaw_link.STL
Joints:
- joint right_hip_pitch_joint: origin xyz=0 0.02605 -0.123 rpy=0 0 0 -> xyz=0 0.026 -0.123 rpy=0 0 0

File: x1_without_skin/urdf/X1.urdf (robot description, URDF)
Before this commit: robot X1, 26 links, 25 joints
Links:
- link head_link: mass 2.6996534 -> 2.717377; geometry collision sphere radius=0.0621; visual mesh filename=../meshes/head_link.STL
- link left_ankle_pitch_link: geometry collision sphere radius=0.035; visual mesh filename=../meshes/left_ankle_pitch_link.STL
- link left_ankle_roll_link: geometry collision sphere radius=0.01; collision sphere radius=0.01
- link left_elbow_link: geometry collision cylinder length=0.08 radius=0.02; visual mesh filename=../meshes/left_elbow_link.STL
- link left_hand_roll_link: geometry collision cylinder length=0.2 radius=0.02; visual mesh filename=../meshes/left_hand_roll_link.STL
- link left_hip_pitch_link: geometry collision cylinder length=0.3 radius=0.05; visual mesh filename=../meshes/left_hip_pitch_link.STL
- link left_hip_roll_link: geometry collision sphere radius=0.04; visual mesh filename=../meshes/left_hip_roll_link.STL
- link left_hip_yaw_link: geometry collision sphere radius=0.05; visual mesh filename=../meshes/left_hip_yaw_link.STL
- link left_knee_link: geometry collision cylinder length=0.25 radius=0.05; visual mesh filename=../meshes/left_knee_link.STL
- link left_shoulder_pitch_link: geometry collision sphere radius=0.025; visual mesh filename=../meshes/left_shoulder_pitch_link.STL
- link left_shoulder_roll_link: geometry collision cylinder length=0.1 radius=0.02; visual mesh filename=../meshes/left_shoulder_roll_link.STL
- link left_shoulder_yaw_link: geometry collision cylinder length=0.07 radius=0.02; visual mesh filename=../meshes/left_shoulder_yaw_link.STL
- link pelvis_link: geometry visual mesh filename=../meshes/pelvis_link.STL
- link right_ankle_pitch_link: geometry collision sphere radius=0.035; visual mesh filename=../meshes/right_ankle_pitch_link.STL
- link right_ankle_roll_link: geometry collision sphere radius=0.01; collision sphere radius=0.01
- link right_elbow_link: geometry collision cylinder length=0.08 radius=0.02; visual mesh filename=../meshes/right_elbow_link.STL
- link right_hand_roll_link: geometry collision cylinder length=0.2 radius=0.02; visual mesh filename=../meshes/right_hand_roll_link.STL
- link right_hip_pitch_link: geometry collision cylinder length=0.3 radius=0.05; visual mesh filename=../meshes/right_hip_pitch_link.STL
- link right_hip_roll_link: geometry collision sphere radius=0.04; visual mesh filename=../meshes/right_hip_roll_link.STL
- link right_hip_yaw_link: geometry collision sphere radius=0.05; visual mesh filename=../meshes/right_hip_yaw_link.STL
- link right_knee_link: geometry collision cylinder length=0.25 radius=0.05; visual mesh filename=../meshes/right_knee_link.STL
- link right_shoulder_pitch_link: geometry collision sphere radius=0.025; visual mesh filename=../meshes/right_shoulder_pitch_link.STL
- link right_shoulder_roll_link: geometry collision cylinder length=0.1 radius=0.02; visual mesh filename=../meshes/right_shoulder_roll_link.STL
- link right_shoulder_yaw_link: geometry collision cylinder length=0.07 radius=0.02; visual mesh filename=../meshes/right_shoulder_yaw_link.STL
- link torso_link: geometry collision cylinder length=0.3 radius=0.1; visual mesh filename=../meshes/torso_link.STL
- link waist_yaw_link: geometry visual mesh filename=../meshes/waist_yaw_link.STL
Joints:
- joint right_hip_pitch_joint: origin xyz=0 0.02605 -0.123 rpy=0 0 0 -> xyz=0 0.026 -0.123 rpy=0 0 0

Commit message: 碰撞体优化

File: x1_with_skin/urdf/X1.urdf (robot description, URDF)
Before this commit: robot X1, 26 links, 25 joints
Links:
- link head_link: geometry collision sphere radius=0.08; visual mesh filename=../meshes/head_link.STL
- link left_ankle_roll_link: geometry collision sphere radius=0.008; collision sphere radius=0.008
- link right_ankle_roll_link: geometry collision sphere radius=0.008; collision sphere radius=0.008
- link torso_link: geometry collision cylinder length=0.35 radius=0.09; visual mesh filename=../meshes/torso_link.STL

File: x1_without_skin/urdf/X1.urdf (robot description, URDF)
Before this commit: robot X1, 26 links, 25 joints
Links:
- link head_link: geometry collision sphere radius=0.08; visual mesh filename=../meshes/head_link.STL
- link left_ankle_roll_link: geometry collision sphere radius=0.008; collision sphere radius=0.008
- link right_ankle_roll_link: geometry collision sphere radius=0.008; collision sphere radius=0.008
- link torso_link: geometry collision cylinder length=0.35 radius=0.09; visual mesh filename=../meshes/torso_link.STL
